Commit message: Updated code with new changes to the robot, also the first step of adding lidar to the base

File: urdf/general_properties.urdf.xacro (robot description, xacro)
@@ -2,8 +2,8 @@
 <robot xmlns:xacro="http://www.ros.org/wiki/xacro">
   <material name="yellow">
-    <color rgba="1 1 0 0.9" />
+    <color rgba="1 1 0 1" />
   </material>
-  <material name="grey">
-    <color rgba="1 1 1 1" />
+  <material name="blue">
+    <color rgba="0.27 0.6 0.9 0.9" />
   </material>
   <xacro:macro name="box_inertia" params="m x y z o_xyz o_rpy">
@@ -25,3 +25,12 @@
     </inertial>
   </xacro:macro>
+  <xacro:macro name="sphere_inertia" params="m r o_xyz o_rpy">
+    <inertial>
+      <mass value="${m}" />
+      <origin xyz="${o_xyz}" rpy="${o_rpy}" />
+      <inertia ixx="${(2/5)*m*r*r}" ixy="0" ixz="0"
+               iyy="${(2/5)*m*r*r}" iyz="0"
+               izz="${(2/5)*m*r*r}" />
+    </inertial>
+  </xacro:macro>
 </robot>

File: urdf/mobile_base.urdf.xacro (robot description, xacro)
@@ -1,9 +1,9 @@
 <?xml version="1.0"?>
 <robot xmlns:xacro="http://www.ros.org/wiki/xacro">
-  <xacro:property name="base_length" value="1.2" />
-  <xacro:property name="base_width" value="0.8" />
+  <xacro:property name="base_length" value="2" />
+  <xacro:property name="base_width" value="1.5" />
   <xacro:property name="base_height" value="0.4" />
-  <xacro:property name="wheel_radius" value="${(base_height * (3/4)) / 2}" />
-  <xacro:property name="wheel_length" value="0.05" />
+  <xacro:property name="wheel_radius" value="${(base_height * (4/4)) / 2}" />
+  <xacro:property name="wheel_length" value="0.2" />
   <link name="base_link">
     <visual>
@@ -12,5 +12,5 @@
       </geometry>
       <origin xyz="0 0 ${base_height / 2.0}" rpy="0 0 0" />
-      <material name="yellow" />
+      <material name="blue" />
     </visual>
     <collision>
@@ -30,5 +30,5 @@
         </geometry>
         <origin xyz="0 0 0" rpy="${pi / 2.0} 0 0" />
-        <material name="grey" />
+        <material name="yellow" />
       </visual>
       <collision>
@@ -44,8 +44,28 @@
   <xacro:wheel_link prefix="right_back" />
   <xacro:wheel_link prefix="left_back" />
-  <xacro:wheel_link prefix="right_front" />
-  <xacro:wheel_link prefix="left_front" />
   <link name="base_footprint">
   </link>
+  <link name="front_wheel_link">
+    <visual>
+      <geometry>
+        <sphere radius="${wheel_radius}" />
+      </geometry>
+      <origin xyz="0 0 0" rpy="0 0 0" />
+      <material name="yellow" />
+    </visual>
+    <collision>
+      <geometry>
+        <sphere radius="${wheel_radius}" />
+      </geometry>
+      <origin xyz="0 0 0" rpy="0 0 0" />
+    </collision>
+    <xacro:sphere_inertia m="2" r="${wheel_radius}"
+                          o_xyz="0 0 0" o_rpy="0 0 0" />
+  </link>
+  <joint name="base_front_wheel_joint" type="fixed">
+    <parent link="base_link" />
+    <child link="front_wheel_link" />
+    <origin xyz="${base_length / 2.6} 0 0" rpy="0 0 0" />
+  </joint>
   <joint name="base_right_back_wheel_joint" type="continuous">
     <parent link="base_link" />
@@ -60,20 +80,8 @@
     <axis xyz="0 1 0" />
   </joint>
-  <joint name="base_right_front_wheel_joint" type="continuous">
-    <parent link="base_link" />
-    <child link="right_front_wheel_link" />
-    <origin xyz="${base_length / 3.0} ${-base_width / 2.0} 0" rpy="0 0 0" />
-    <axis xyz="0 1 0" />
-  </joint>
-  <joint name="base_left_front_wheel_joint" type="continuous">
-    <parent link="base_link" />
-    <child link="left_front_wheel_link" />
-    <origin xyz="${base_length / 3.0} ${base_width / 2.0} 0" rpy="0 0 0" />
-    <axis xyz="0 1 0" />
-  </joint>
   <joint name="base_joint" type="fixed">
     <parent link="base_footprint" />
     <child link="base_link" />
-    <origin xyz="0 0 ${(base_height * (3/4)) / 2}" rpy="0 0 0" />
+    <origin xyz="0 0 ${(base_height * (4/4)) / 2}" rpy="0 0 0" />
     <axis xyz="0 0 0" />
   </joint>

File: urdf/my_robot.urdf.xacro (robot description, xacro)
@@ -3,3 +3,5 @@
   <xacro:include filename="general_properties.urdf.xacro" />
   <xacro:include filename="mobile_base.urdf.xacro" />
+  <xacro:include filename="mobile_base_gazebo.urdf.xacro" />
+  <xacro:include filename="lidar.urdf.xacro" />
 </robot>
