Commit message: Polished files, removed uneccessary code

File: my_robot_description/urdf/lidar.urdf.xacro (robot description, xacro)
@@ -3,5 +3,5 @@
   <xacro:property name="lidar_radius" value="0.1" />
   <xacro:property name="lidar_length" value="0.1" />
-  <link name="lidar_scanner_link">
+  <link name="lidar_link">
     <visual>
       <geometry>
@@ -19,8 +19,8 @@
                             o_xyz="0 0 0" o_rpy="${pi / 2.0} 0 0" />
   </link>
-  <joint name="base_lidar_scanner_joint" type="fixed">
+  <joint name="base_lidar_joint" type="fixed">
     <parent link="base_link" />
-    <child link="lidar_scanner_link" />
-    <origin xyz="0 0 ${base_height}" rpy="0 0 0" />
+    <child link="lidar_link" />
+    <origin xyz="0 0 ${base_height + (1/2) * lidar_length}" rpy="0 0 0" />
   </joint>
 </robot>

File: my_robot_description/urdf/mobile_base.urdf.xacro (robot description, xacro)
@@ -83,5 +83,5 @@
     <parent link="base_footprint" />
     <child link="base_link" />
-    <origin xyz="0 0 ${(base_height * (4/4)) / 2}" rpy="0 0 0" />
+    <origin xyz="${base_length / 3.0} 0 ${(base_height * (4/4)) / 2}" rpy="0 0 0" />
     <axis xyz="0 0 0" />
   </joint>

File: my_robot_description/urdf/mobile_base_gazebo.urdf.xacro (robot description, xacro)
@@ -17,7 +17,49 @@
       <wheel_separation>1.5</wheel_separation>
       <wheel_radius>0.2</wheel_radius>
+      <topic>/cmd_vel</topic>
+      <tf_topic>/tf</tf_topic>
+      <odom_topic>/odom</odom_topic>
       <frame_id>odom</frame_id>
       <child_frame_id>base_footprint</child_frame_id>
+      <publish_odom>true</publish_odom>
+      <publish_tf>true</publish_tf>
+      <odom_publisher_frequency>30</odom_publisher_frequency>
     </plugin>
   </gazebo>
+  <gazebo>
+    <plugin filename="gz-sim-sensors-system" name="gz::sim::systems::Sensors">
+      <render_engine>ogre2</render_engine>
+    </plugin>
+  </gazebo>
+  <gazebo reference="lidar_link">
+    <sensor name="gpu_lidar" type="gpu_lidar">
+      <pose relative_to="lidar_link">0 0 0 0 0 0</pose>
+      <topic>scan</topic>
+      <gz_frame_id>lidar_link</gz_frame_id>
+      <frame_id>lidar_link</frame_id>
+      <always_on>true</always_on>
+      <visualize>true</visualize>
+      <update_rate>20</update_rate>
+      <lidar>
+        <scan>
+          <horizontal>
+            <samples>720</samples>
+            <resolution>1.0</resolution>
+            <min_angle>-3.14</min_angle>
+            <max_angle>3.14</max_angle>
+          </horizontal>
+        </scan>
+        <range>
+          <min>0.4</min>
+          <max>10.0</max>
+          <resolution>0.001</resolution>
+        </range>
+        <noise>
+          <type>gaussian</type>
+          <mean>0.0</mean>
+          <stddev>0.001</stddev>
+        </noise>
+      </lidar>
+    </sensor>
+  </gazebo>
 </robot>

File: my_robot_description/urdf/my_robot.urdf.xacro (robot description, xacro)
@@ -3,5 +3,5 @@
   <xacro:include filename="general_properties.urdf.xacro" />
   <xacro:include filename="mobile_base.urdf.xacro" />
+   <xacro:include filename="lidar.urdf.xacro" />
   <xacro:include filename="mobile_base_gazebo.urdf.xacro" />
-  <xacro:include filename="lidar.urdf.xacro" />
 </robot>
